File: ez_rail.kicad_pcb (KiCad board)
At the start: 2 copper layers, 16 parts, among them J1 Conn_01x02_Male, J2 Conn_01x02_Male, J3 Conn_01x03_Male, U1 LM2575T, U2 LM2575T

Commit message: Finishing layout, adding gitignore, removing cache file
Adding media & readme
Parts:
- removed J1, J2: Conn_01x02_Male, Connector_PinHeader_2.54mm:PinHeader_1x02_P2.54mm_Vertical
- removed R1, R2: 1R, Resistor_THT:R_Axial_DIN0614_L14.3mm_D5.7mm_P15.24mm_Horizontal
- moved J3 46.1 mm to (133.1, 106.1), turned to 90 degrees
Connections:
- J3 pad 2: Net-(J2-Pad2) -> +5V
- J3 pad 3: Net-(J1-Pad2) -> +3V3
Routing:
- net +9V: track 0.00 -> 58.0 mm
- net +5V: track 0.00 -> 41.1 mm
- net +3V3: track 0.00 -> 39.2 mm
- net Net-(D1-Pad1): track 0.00 -> 17.5 mm
- net Net-(D2-Pad1): track 0.00 -> 15.4 mm
- net GND: track 0.00 -> 5.24 mm
- added copper zone on B.Cu, net GND
Other:
- board outline added: 56 x 30 mm
